File: Output_Amp.kicad_sch (KiCad schematic)
At the start: 5 parts, among them U5 OPA1679

Commit message: Version 1 ready to order
Parts:
- R1101: LCSC (none) -> C4184
- R1102: LCSC (none) -> C25808
- R1103: LCSC (none) -> C21190
- U5: LCSC (none) -> C2057264
Changed lines of the file:
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@@
 		(shape input)
 		(at 167.64 128.27 180)
-		(fields_autoplaced yes)
 		(effects
 			(font
@@
 		(shape output)
 		(at 218.44 128.27 0)
-		(fields_autoplaced yes)
 		(effects
 			(font
@@
 			)
 		)
+		(property "LCSC" " C21190"
+			(at 210.82 128.27 0)
+			(effects
+				(font
+					(size 1.27 1.27)
+				)
+				(hide yes)
+			)
+		)
 		(pin "2"
 		)
@@
 		(property "MPN" "OPA1679"
 			(at 199.39 146.05 0)
+			(effects
+				(font
+					(size 1.27 1.27)
+				)
+				(hide yes)
+			)
+		)
+		(property "LCSC" "C2057264"
+			(at 193.04 138.43 0)
 			(effects
 				(font
@@
 			)
 		)
+		(property "LCSC" "C25808"
+			(at 194.31 128.27 0)
+			(effects
+				(font
+					(size 1.27 1.27)
+				)
+				(hide yes)
+			)
+		)
 		(pin "2"
 		)
@@
 			(at 176.53 128.27 0)
 			(effects
+				(font
+					(size 1.27 1.27)
+				)
+				(hide yes)
+			)
+		)
+		(property "LCSC" " C4184"
+			(at 176.53 128.27 0)
+			(effects
