File: _autosave-Loom_AK4619.kicad_pcb (KiCad board)
At the start: 2 copper layers, 110 x 110 mm, 195 parts, among them J1 Conn_01x40, J2 Conn_01x40, U1 AK4619VN, U101 HT75xx-1-SOT89, U2 AK4619VN, U3 OPA1679, U4 OPA1679, U5 OPA1679, U6 OPA1679

Commit message: Version 1 ready to order
Other:
- board text added: "Loom AK4619 V1 Carson Walls 2/2025"
- board text removed: "Loom AK4619 Carson Walls 2/2025"
Changed lines of the file:
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@@
 		)
 	)
-	(gr_text "Loom AK4619\nCarson Walls\n2/2025"
+	(gr_text "Loom AK4619 V1\nCarson Walls\n2/2025"
 		(at 125.147 111.841 90)
 		(layer "F.SilkS")
